File: analog-frontend.brd (EAGLE design)
At the start: 28.4 x 25.2 mm, 69 parts, among them IC1 TPS63031, IC2 ADG731, IC3 TM4C123G, IC4 INA332, IC5 NRF24L01SMD, IC6 OPA2320, Y1 CRYSTAL3X2, Y2 CRYSTAL3X2

Commit message: almost final board files
Parts:
- removed TP1, TP2, TP3, TP4, TP5, TP6, TP7, TP8, TP9: PTR1B1,27, testpad:B1,27
- added 3.3V, GND, RST, RXD, TCK, TDI, TDO, TMS, TXD: PTR1B1,27, testpad:B1,27
- C4, C7: device rcl:C0201 -> rcl:C0402
- moved U$1 1.01 mm to (26.8, 15.6)
- moved C20 0.81 mm to (21.6, 11.7)
- moved C19 0.79 mm to (19.0, 21.4)
- moved C22 0.79 mm to (23.7, 16.1)
- moved C23 0.79 mm to (19.9, 14.2)
- moved C26 0.79 mm to (24.3, 20.4)
- moved C28 0.79 mm to (26.5, 8.32)
- moved C3 0.79 mm to (22.6, 6.40)
- moved C6 0.79 mm to (18.1, 13.8)
- moved JP1 0.79 mm to (26.2, 3.92)
- moved JP2 0.79 mm to (26.2, 1.65)
- moved JP3 0.79 mm to (26.2, 23.5)
- moved L1 0.79 mm to (19.7, 8.12)
- moved L2 0.79 mm to (23.5, 18.6)
- moved L4 0.79 mm to (24.8, 16.5)
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Connections:
- net +3V3: now also 3.3V.TP; no longer TP8.TP
- net GND: now also GND.TP; no longer TP9.TP
- net N$49: now also RST.TP; no longer TP7.TP
- net RXD: now also RXD.TP; no longer TP1.TP
- net TCK: now also TCK.TP; no longer TP3.TP
- net TDI: now also TDI.TP; no longer TP5.TP
- net TDO: now also TDO.TP; no longer TP6.TP
- net TMS: now also TMS.TP; no longer TP4.TP
- net TXD: now also TXD.TP; no longer TP2.TP
Routing:
- net +3V3: track 114.9 -> 116.1 mm
- net VCM1: track 11.2 -> 11.9 mm
- net VDDA: track 73.5 -> 74.2 mm
- net GNDA: track 93.3 -> 92.7 mm
Other:
- board text added: "+"
