File: analog-frontend.sch (EAGLE design)
At the start: 69 parts, among them IC1 TPS63031, IC2 ADG731, IC3 TM4C123G, IC4 INA332, IC5 NRF24L01SMD, IC6 OPA2320, Y1 CRYSTAL3X2, Y2 CRYSTAL3X2

Commit message: minor changes
Parts:
- added R16: (no value), FAB_Hello:RESISTOR0402
Connections:
- removed net N$41: C28.1, IC6.OUTB, R12.1
- new net AIN: C28.1, IC5.PB5, IC6.OUTB, R12.1
Changed lines of the file:
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@@
 <part name="R3" library="rcl" deviceset="R-US_" device="R0402"/>
 <part name="SUPPLY25" library="supply2" deviceset="GND" device=""/>
+<part name="R16" library="FAB_Hello" deviceset="RESISTOR" device="0402"/>
 </parts>
 <sheets>
@@
 <instance part="R3" gate="G$1" x="149.86" y="68.58" rot="R90"/>
 <instance part="SUPPLY25" gate="GND" x="149.86" y="55.88"/>
+<instance part="R16" gate="G$1" x="116.84" y="149.86"/>
 </instances>
 <busses>
@@
 </segment>
 </net>
-<net name="N$41" class="0">
+<net name="AIN" class="0">
 <segment>
 <pinref part="R12" gate="G$1" pin="1"/>
@@
 <wire x1="340.36" y1="233.68" x2="340.36" y2="226.06" width="0.1524" layer="91"/>
 <junction x="340.36" y="226.06"/>
-</segment>
-</net>
+<wire x1="340.36" y1="233.68" x2="340.36" y2="241.3" width="0.1524" layer="91"/>
+<junction x="340.36" y="233.68"/>
+<wire x1="340.36" y1="241.3" x2="342.9" y2="241.3" width="0.1524" layer="91"/>
+<label x="342.9" y="241.3" size="1.27" layer="95" xref="yes"/>
+</segment>
+<segment>
+<pinref part="IC5" gate="A" pin="PB5"/>
+<wire x1="213.36" y1="121.92" x2="220.98" y2="121.92" width="0.1524" layer="91"/>
+<label x="220.98" y="121.92" size="1.27" layer="95" xref="yes"/>
+</segment>
+</net>
