File: connector-32ch.brd (EAGLE design)
At the start: 26.7 x 25.1 mm, 67 parts, among them X1 OMNETICS_36PAD

Commit message: almost final board files
Parts:
- C1, C10, C11, C12, C13, C14, C15, C16, C17, C18, C19, C2, C20, C21, C22, C23, C24, C25, C26, C27, C28, C29, C3, C30, C31, C32, C4, C5, C6, C7, C8, C9: value (none) -> 22nf
- X1: device mor307:OMNETICS36PADPTH -> mor307:OMNETICS36PADSMT
- moved X1 0.63 mm to (13.3, 12.7)
- flipped C1 to the bottom
- flipped C10 to the bottom
- flipped C11 to the bottom
- flipped C12 to the bottom
- flipped C13 to the bottom
- flipped C14 to the bottom
- flipped C15 to the bottom
- flipped C16 to the bottom
- flipped C17 to the bottom
- flipped C18 to the bottom
- flipped C19 to the bottom
- flipped C2 to the bottom
- flipped C20 to the bottom
- flipped C21 to the bottom
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Connections:
- net G: now also JP1.2, X1.R1; no longer JP1.19, X1.G1
- net R: now also JP1.19, X1.G1; no longer JP1.2, X1.R1
Routing:
- net G: track 26.2 -> 45.0 mm, vias 0 -> 2
- net R: track 26.2 -> 42.8 mm, vias 0 -> 2
- added copper zone on layer 16, net G
- added copper zone on layer 1, net VCM
- removed copper zone on layer 1, net G
- removed copper zone on layer 1, net R
- removed copper zone on layer 16, net VCM

Commit message: added component values
Other:
- board outline removed
Changed lines of the file:
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@@
 <?xml version="1.0" encoding="utf-8"?>
 <!DOCTYPE eagle SYSTEM "eagle.dtd">
-<eagle version="6.5.0">
+<eagle version="6.6.0">
 <drawing>
 <settings>
@@
 <setting verticaltext="up"/>
 </settings>
-<grid distance="0.0025" unitdist="inch" unit="inch" style="lines" multiple="1" display="yes" altdistance="0.025" altunitdist="inch" altunit="inch"/>
+<grid distance="0.001" unitdist="inch" unit="inch" style="lines" multiple="1" display="yes" altdistance="0.025" altunitdist="inch" altunit="inch"/>
 <layers>
 <layer number="1" name="Top" color="4" fill="1" visible="yes" active="yes"/>
@@
 <board>
 <plain>
-<wire x1="0" y1="0" x2="26.67" y2="0" width="0" layer="20"/>
-<wire x1="26.67" y1="0" x2="26.67" y2="25.146" width="0" layer="20"/>
-<wire x1="26.67" y1="25.146" x2="0" y2="25.146" width="0" layer="20"/>
-<wire x1="0" y1="25.146" x2="0" y2="0" width="0" layer="20"/>
+<wire x1="0" y1="0" x2="26.67" y2="0" width="0" layer="21"/>
+<wire x1="26.67" y1="0" x2="26.67" y2="25.146" width="0" layer="21"/>
+<wire x1="26.67" y1="25.146" x2="0" y2="25.146" width="0" layer="21"/>
+<wire x1="0" y1="25.146" x2="0" y2="0" width="0" layer="21"/>
 <text x="2.159" y="22.5425" size="0.8128" layer="25" rot="R270">GND</text>
 <text x="2.8575" y="2.7305" size="0.8128" layer="25" font="fixed" rot="R90">REF</text>
@@
 <text x="23.8125" y="22.4155" size="0.8128" layer="25" font="fixed" rot="R270">REF</text>
 <rectangle x1="24.9047" y1="2.7686" x2="25.7683" y2="5.3594" layer="25"/>
+<wire x1="0" y1="0" x2="26.67" y2="0" width="0" layer="22"/>
+<wire x1="26.67" y1="0" x2="26.67" y2="25.146" width="0" layer="22"/>
+<wire x1="26.67" y1="25.146" x2="0" y2="25.146" width="0" layer="22"/>
+<wire x1="0" y1="25.146" x2="0" y2="0" width="0" layer="22"/>
 </plain>
 <attributes>
